Commit message: 该分支含rtk相关

File: buaahz_car_urdf_Mid360/urdf/buaahz_car_urdf_mid360.urdf (robot description, URDF)
Before this commit: robot buaahz_car_urdf_mid360, 9 links, 8 joints
Links:
- link lidar_link: mass 0.14188701649649 -> 0.141887205117604
Joints:
- joint lidar_joint: origin xyz=0.2528 -0.049062 1.3221 rpy=3.1416 0 0 -> xyz=0.2528 -0.0001 1.3221 rpy=3.1416 0 0
- joint rf_joint: origin xyz=0.3818 -0.17625 0.0052475 rpy=0 0 0 -> xyz=0.3818 0.17675 0.0052475 rpy=0 0 0
- joint rf_wheel_joint: origin xyz=-0.024001 0 -0.055747 rpy=0 0 0 -> xyz=-0.024001 -0.353 -0.055747 rpy=0 0 0

File: buaahz_car_urdf_Mid360/urdf/g1_urdf.urdf (robot description, URDF)
Before this commit: robot two_link_robot, 2 links, 1 joints
Links:
- added link gps_link, mass 0.5; collision cylinder length=0.2 radius=0.1; visual cylinder length=0.2 radius=0.1
Joints:
- added joint base_to_gps_joint: type fixed, parent base_link, child gps_link, origin xyz=0 0 0.28 rpy=0 3.14 3.14, limit effort=1000.0 velocity=1000.0

Commit message: 添加ultrasoud link

File: buaahz_car_urdf_Mid360/urdf/buaahz_car_urdf_mid360.urdf (robot description, URDF)
Before this commit: robot buaahz_car_urdf_mid360, 9 links, 8 joints
Links:
- added link ultrasound_link1, mass 0.00233498324559951; collision mesh filename=package://buaahz_car_urdf_mid360/meshes/ultrasound_link1.STL; visual mesh filename=package://buaahz_car_urdf_mid360/meshes/ultrasound_link1.STL
- added link ultrasound_link2, mass 0.00233498324559952; collision mesh filename=package://buaahz_car_urdf_mid360/meshes/ultrasound_link2.STL; visual mesh filename=package://buaahz_car_urdf_mid360/meshes/ultrasound_link2.STL
- added link ultrasound_link3, mass 0.00233498324559954; collision mesh filename=package://buaahz_car_urdf_mid360/meshes/ultrasound_link3.STL; visual mesh filename=package://buaahz_car_urdf_mid360/meshes/ultrasound_link3.STL
- added link ultrasound_link4, mass 0.0023349832455997; collision mesh filename=package://buaahz_car_urdf_mid360/meshes/ultrasound_link4.STL; visual mesh filename=package://buaahz_car_urdf_mid360/meshes/ultrasound_link4.STL
- added link ultrasound_link5, mass 0.00233498324559952; collision mesh filename=package://buaahz_car_urdf_mid360/meshes/ultrasound_link5.STL; visual mesh filename=package://buaahz_car_urdf_mid360/meshes/ultrasound_link5.STL
- added link ultrasound_link6, mass 0.0023349832455996; collision mesh filename=package://buaahz_car_urdf_mid360/meshes/ultrasound_link6.STL; visual mesh filename=package://buaahz_car_urdf_mid360/meshes/ultrasound_link6.STL
- added link ultrasound_link7, mass 0.00233498324559957; collision mesh filename=package://buaahz_car_urdf_mid360/meshes/ultrasound_link7.STL; visual mesh filename=package://buaahz_car_urdf_mid360/meshes/ultrasound_link7.STL
- added link ultrasound_link8, mass 0.00233498324559952; collision mesh filename=package://buaahz_car_urdf_mid360/meshes/ultrasound_link8.STL; visual mesh filename=package://buaahz_car_urdf_mid360/meshes/ultrasound_link8.STL
- link lf_Link: mass 0.0764331852561443 -> 0.0764331852561444
- link lidar_link: mass 0.14188701649649 -> 0.141887208379736
- link rf_Link: mass 0.0764331852561442 -> 0.0764331852561443
Joints:
- added joint ultrasound_joint1: type fixed, parent base_link, child ultrasound_link1, origin xyz=0.4465 0.234 0.069062 rpy=0 0 0, axis 0 0 0
- added joint ultrasound_joint2: type fixed, parent base_link, child ultrasound_link2, origin xyz=0.4465 -0.234 0.069062 rpy=0 0 0, axis 0 0 0
- added joint ultrasound_joint3: type fixed, parent base_link, child ultrasound_link3, origin xyz=0.3375 -0.274 0.069062 rpy=0 0 -1.5708, axis 0 0 0
- added joint ultrasound_joint4: type fixed, parent base_link, child ultrasound_link4, origin xyz=0.0075 -0.274 0.069062 rpy=0 0 -1.5708, axis 0 0 0
- added joint ultrasound_joint5: type fixed, parent base_link, child ultrasound_link5, origin xyz=-0.1015 -0.234 0.069062 rpy=0 0 3.1416, axis 0 0 0
- added joint ultrasound_joint7: type fixed, parent base_link, child ultrasound_link7, origin xyz=0.0075 0.274 0.069062 rpy=0 0 1.5708, axis 0 0 0
- added joint ultrasound_joint8: type fixed, parent base_link, child ultrasound_link8, origin xyz=0.3175 0.274 0.049 rpy=-1.5708 3.14159 -1.5708, axis 0 0 0
- added joint ultrasound_link6: type fixed, parent base_link, child ultrasound_link6, origin xyz=-0.1015 0.234 0.069062 rpy=0 0 -3.1416, axis 0 0 0
- joint lidar_joint: origin xyz=0.2528 -0.049062 1.3221 rpy=3.1416 0 0 -> xyz=0.2522 0.0001 1.3221 rpy=3.1416 0 0

Commit message: 保持与main分支一致

File: buaahz_car_urdf_Mid360/urdf/buaahz_car_urdf_mid360.urdf (robot description, URDF)
Before this commit: robot buaahz_car_urdf_mid360, 9 links, 8 joints
Links:
- added link ultrasound_link1, mass 0.00233498324559951; collision mesh filename=package://buaahz_car_urdf_mid360/meshes/ultrasound_link1.STL; visual mesh filename=package://buaahz_car_urdf_mid360/meshes/ultrasound_link1.STL
- added link ultrasound_link2, mass 0.00233498324559952; collision mesh filename=package://buaahz_car_urdf_mid360/meshes/ultrasound_link2.STL; visual mesh filename=package://buaahz_car_urdf_mid360/meshes/ultrasound_link2.STL
- added link ultrasound_link3, mass 0.00233498324559954; collision mesh filename=package://buaahz_car_urdf_mid360/meshes/ultrasound_link3.STL; visual mesh filename=package://buaahz_car_urdf_mid360/meshes/ultrasound_link3.STL
- added link ultrasound_link4, mass 0.0023349832455997; collision mesh filename=package://buaahz_car_urdf_mid360/meshes/ultrasound_link4.STL; visual mesh filename=package://buaahz_car_urdf_mid360/meshes/ultrasound_link4.STL
- added link ultrasound_link5, mass 0.00233498324559952; collision mesh filename=package://buaahz_car_urdf_mid360/meshes/ultrasound_link5.STL; visual mesh filename=package://buaahz_car_urdf_mid360/meshes/ultrasound_link5.STL
- added link ultrasound_link6, mass 0.0023349832455996; collision mesh filename=package://buaahz_car_urdf_mid360/meshes/ultrasound_link6.STL; visual mesh filename=package://buaahz_car_urdf_mid360/meshes/ultrasound_link6.STL
- added link ultrasound_link7, mass 0.00233498324559957; collision mesh filename=package://buaahz_car_urdf_mid360/meshes/ultrasound_link7.STL; visual mesh filename=package://buaahz_car_urdf_mid360/meshes/ultrasound_link7.STL
- added link ultrasound_link8, mass 0.00233498324559952; collision mesh filename=package://buaahz_car_urdf_mid360/meshes/ultrasound_link8.STL; visual mesh filename=package://buaahz_car_urdf_mid360/meshes/ultrasound_link8.STL
- link lf_Link: mass 0.0764331852561443 -> 0.0764331852561444
- link lidar_link: mass 0.141887205117604 -> 0.141887208379736
- link rf_Link: mass 0.0764331852561442 -> 0.0764331852561443
Joints:
- added joint ultrasound_joint1: type fixed, parent base_link, child ultrasound_link1, origin xyz=0.4465 0.234 0.069062 rpy=0 0 0, axis 0 0 0
- added joint ultrasound_joint2: type fixed, parent base_link, child ultrasound_link2, origin xyz=0.4465 -0.234 0.069062 rpy=0 0 0, axis 0 0 0
- added joint ultrasound_joint3: type fixed, parent base_link, child ultrasound_link3, origin xyz=0.3375 -0.274 0.069062 rpy=0 0 -1.5708, axis 0 0 0
- added joint ultrasound_joint4: type fixed, parent base_link, child ultrasound_link4, origin xyz=0.0075 -0.274 0.069062 rpy=0 0 -1.5708, axis 0 0 0
- added joint ultrasound_joint5: type fixed, parent base_link, child ultrasound_link5, origin xyz=-0.1015 -0.234 0.069062 rpy=0 0 3.1416, axis 0 0 0
- added joint ultrasound_joint7: type fixed, parent base_link, child ultrasound_link7, origin xyz=0.0075 0.274 0.069062 rpy=0 0 1.5708, axis 0 0 0
- added joint ultrasound_joint8: type fixed, parent base_link, child ultrasound_link8, origin xyz=0.3175 0.274 0.049 rpy=-1.5708 3.14159 -1.5708, axis 0 0 0
- added joint ultrasound_link6: type fixed, parent base_link, child ultrasound_link6, origin xyz=-0.1015 0.234 0.069062 rpy=0 0 -3.1416, axis 0 0 0
- joint lidar_joint: origin xyz=0.2528 -0.0001 1.3221 rpy=3.1416 0 0 -> xyz=0.2522 0.0001 1.3221 rpy=3.1416 0 0
- joint rf_joint: origin xyz=0.3818 0.17675 0.0052475 rpy=0 0 0 -> xyz=0.3818 -0.17625 0.0052475 rpy=0 0 0
- joint rf_wheel_joint: origin xyz=-0.024001 -0.353 -0.055747 rpy=0 0 0 -> xyz=-0.024001 0 -0.055747 rpy=0 0 0

Commit message: gengxin

File: buaahz_car_urdf_Mid360/urdf/buaahz_car_urdf_mid360.urdf (robot description, URDF)
Before this commit: robot buaahz_car_urdf_mid360, 17 links, 16 joints
Links:
- added link gps_link, mass 0.1; collision box size=0.08 0.08 0.04; visual box size=0.08 0.08 0.04
Joints:
- added joint base_link_to_gps_link: type fixed, parent base_link, child gps_link, origin xyz=0 0 0 rpy=0 0 -2.335

Commit message: gengxin

File: buaahz_car_urdf_Mid360/urdf/buaahz_car_urdf_mid360.urdf (robot description, URDF)
Before this commit: robot buaahz_car_urdf_mid360, 18 links, 17 joints
Joints:
- joint base_link_to_gps_link: origin xyz=0 0 0 rpy=0 0 -2.335 -> xyz=0.2 -0.17 1.25 rpy=0 0 0
